File: Schema/Schema.kicad_sch (KiCad schematic)
At the start: 4 parts

Commit message: schema electrique
Parts:
- removed J?: XLR3_Switched, symbol Connector:XLR3_Switched
- removed U?: 74LS46, symbol 74xx:74LS46
- added 7Seg1, 7Seg2: 7 segment, symbol Display_Character:HDSP-7801
- added Bouton?: BP_Prog_Etat_Apres_Valide, symbol Switch:SW_Push
- added Bouton?: BP_Prog_Direction_SW, symbol Switch:SW_Push
- added Bouton?: BP_Prog_Bouton_Lancer_Principale, symbol Switch:SW_Push
- added Bouton?: BP_Prog_Etat_Avant_Letter, symbol Switch:SW_Push
- added Bouton?: BP_Prog_Ecran_LCD_Moins, symbol Switch:SW_Push
- added Bouton?: BP_Prog_Ecran_LCD_Plus, symbol Switch:SW_Push
- added Bouton?: BP_Prog_Etat_Avant_Valide, symbol Switch:SW_Push
- added Bouton?: BP_Prog_Ruban_LED_Change_Letter, symbol Switch:SW_Push
- added Bouton?: BP_Prog_Ruban_LED_Valid_Letter, symbol Switch:SW_Push
- added Bouton?: BP_Prog_Etat_Avant_Plus, symbol Switch:SW_Push
- added Bouton?: BP_Prog_Etat_Apres_Moins, symbol Switch:SW_Push
- added Bouton?: BP_Prog_Ecran_LCD_Valide, symbol Switch:SW_Push
- added Bouton?: BP_Prog_Etat_Avant_Moins, symbol Switch:SW_Push
- added Bouton?: BP_Prog_Etat_Apres_Plus, symbol Switch:SW_Push
- added D?: LED_Etat_Apres, symbol Device:LED_RGBK
- added D?: LED_Etat_Avant_Letter, symbol Device:LED_RGBK
- added D?: LED_Direction_Gauche, symbol Device:LED
- added D?: LED_Direction_Droite, symbol Device:LED
- added R, R? (x13): 120, symbol Device:R
- added R? (x16): 10k, symbol Device:R
- added R? (x3): 4.7k, symbol Device:R
- added R?: ?, symbol Device:R
- added U?: Expender 2, symbol Interface_Expansion:MCP23017_SO
- added U?: Expender 1, symbol Interface_Expansion:MCP23017_SO
- added U?: Ecran LCD, Display:NHD-C0220BiZ, symbol Display_Character:NHD-C0220BIZ
- added U?: Expender 3, symbol Interface_Expansion:MCP23017_SO
- J?: value XLR3_Switched -> Levier
Connections:
- net +3.3V: now reaches U=5V.13 (VDD)
- net +3.3V: now also U=5V.28 (VDD), Bouton?.1, Bouton?.1, Bouton?.1, Bouton?.1, Bouton?.1, Bouton?.1, Bouton?.1, Bouton?.1, Bouton?.1, Bouton?.1, Bouton?.1, Bouton?.1, Bouton?.1, Bouton?.1, R?.1, R?.1, R?.1, R?.1, R?.1, U?.5 (VDD), U?.9 (VDD), U?.9 (VDD), U?.9 (VDD)
- net SCL1: now reaches U=5V.17 (SCL1)
- net SCL1: now also U?.13 (SDA), U?.13 (SDA), U?.13 (SDA), U?.2 (SCL)
- net SDA1: now reaches U=5V.18 (SDA1)
- net SDA1: now also U?.12 (SCK), U?.12 (SCK), U?.12 (SCK), U?.3 (SDA)
- net Earth: now reaches U=5V.27 (VSS)
- net Earth: now also U=5V.8 (VSS), 7Seg1.5 (VSS), 7Seg2.5 (VSS), D?.1 (K), D?.1 (K), D?.4 (K), D?.4 (K), R?.1, R?.1, R?.1, R?.1, R?.1, R?.1, R?.1, R?.1, R?.1, R?.1, R?.1, R?.1, R?.1, R?.1, U?.10 (VSS), U?.10 (VSS), U?.10 (VSS), U?.15 (A0), U?.16 (A1), U?.17 (A2), U?.17 (A2), U?.17 (A2), U?.4 (VSS)
- new net: R?.2, U?.22 (GPA1)
- new net: R?.2, U?.16 (A1) (x2)
- new net: R?.2, U?.15 (A0) (x2)
- new net: R?.1, U?.7 (GPB6)
- new net: R.1, U?.1 (GPB0)
- new net: R?.2, U?.24 (GPA3)
- new net: R?.1, U?.3 (GPB2)
- new net: R?.2, U?.1 (~{RST})
- new net: R?.1, U?.6 (GPB5)
- new net: D?.1 (RA), R?.2
- new net: R?.2, U?.26 (GPA5)
- new net: R?.1, U?.2 (GPB1)
- new net: R?.2, U?.23 (GPA2)
- new net: R?.2, U?.25 (GPA4)
- new net: R?.2, U?.27 (GPA6)
- new net: R?.2, U?.28 (GPA7)
- new net: R?.1, U?.4 (GPB3)
- new net: R?.1, U?.5 (GPB4)
- new net 7segment_1 A1: 7Seg1.10 (A1), R.2
- new net 7segment_1 B1: 7Seg1.9 (B1), R?.2
- new net 7segment_1 C1: 7Seg1.8 (C1), R?.2
- new net 7segment_1 D1: 7Seg1.7 (D1), R?.2
- new net 7segment_1 E1: 7Seg1.1 (E1), R?.2
- new net 7segment_1 F1: 7Seg1.2 (F1), R?.2
- new net 7segment_1 G1: 7Seg1.3 (G1), R?.2
- new net 7segment_2 A2: 7Seg2.10 (A1), R?.1
- new net 7segment_2 B2: 7Seg2.9 (B1), R?.1
- new net 7segment_2 C2: 7Seg2.8 (C1), R?.1
- new net 7segment_2 D2: 7Seg2.7 (D1), R?.1
- new net 7segment_2 E2: 7Seg2.1 (E1), R?.1
- new net 7segment_2 F2: 7Seg2.2 (F1), R?.1
- new net 7segment_2 G2: 7Seg2.3 (G1), R?.1
- new net BP1: Bouton?.2, Bouton?.2, R?.2, R?.2, U?.1 (GPB0)
- new net BP10: Bouton?.2, R?.2, U?.22 (GPA1)
- new net BP11: Bouton?.2, R?.2, U?.23 (GPA2)
- new net BP12: Bouton?.2, R?.2, U?.24 (GPA3)
- new net BP13: U?.25 (GPA4)
- new net BP14: U?.26 (GPA5)
- new net BP15: Bouton?.2, R?.2, U?.27 (GPA6)
- new net BP16: Bouton?.2, R?.2, U?.28 (GPA7)
- new net BP2: Bouton?.2, R?.2, U?.2 (GPB1)
- new net BP3: U?.3 (GPB2)
- new net BP4: Bouton?.2, R?.2, U?.4 (GPB3)
- new net BP5: Bouton?.2, R?.2, U?.5 (GPB4)
- new net BP6: Bouton?.2, R?.2, U?.6 (GPB5)
- new net BP7: Bouton?.2, R?.2, U?.7 (GPB6)
- new net BP8: Bouton?.2, R?.2, U?.8 (GPB7)
- new net BP9: Bouton?.2, R?.2, U?.21 (GPA0)
- new net LED1: R?.1, U?.1 (GPB0)
- new net LED2: D?.2 (GA), U?.2 (GPB1)
- new net LED3: D?.3 (BA), U?.3 (GPB2)
- new net LED4: D?.2 (A), U?.4 (GPB3)
- new net LED5: D?.2 (A), U?.5 (GPB4)
- new net LED6: D?.1 (RA), U?.6 (GPB5)
- new net LED7: D?.2 (GA), U?.7 (GPB6)
- new net LED8: D?.3 (BA), U?.8 (GPB7)
Other:
- moved on the sheet: J?B, U=5V

Commit message: jcp
Parts:
- added 100nF (x2): Capacitor, symbol Device:C_Small
- added Bouton?: BP_Prog_Ecran_LCD_Plus, symbol Switch:SW_Push
- added D?: LED_Direction_Droite, symbol Device:LED
- added R?: 10k, symbol Device:R
Connections:
- net +3.3V: now also Bouton?.1; no longer U=5V.13 (VDD), U=5V.28 (VDD)
- net BP9: now also Bouton?.2, R?.2
- net Earth: now also D?.1 (K), R?.1; no longer U=5V.27 (VSS), U=5V.8 (VSS)
- net LED_ERREUR: now reaches U=5V.11 (RP4)
- net LED_ERREUR: now also D?.2 (A)
- new net: 100nF.2, U=5V.13 (VDD)
- new net: 100nF.1, U=5V.27 (VSS)
- new net: 100nF.2, U=5V.28 (VDD)
- new net: 100nF.1, U=5V.8 (VSS)
Other:
- moved on the sheet: 7Seg2, U=5V

Commit message: schema finiiii
Parts:
- removed Bouton?: BP_Prog_Ecran_LCD_Plus, symbol Switch:SW_Push
- removed J?: Levier, symbol Connector:XLR3_Switched
- removed R?: 10k, symbol Device:R
- added 100nF?: Capacitor, symbol Device:C_Small
- added HDR1X5: DIN41612_02x05_AB_EvenPins, symbol Connector:DIN41612_02x05_AB_EvenPins
- added ModeContinue/PasAPas?: Levier, symbol Connector:XLR3_Switched
- added R?: 10k, symbol Device:R
- added R?: 200, symbol Device:R
- added U? (x6): Ruban LED, symbol Driver_LED:HV9931LG-G
- Bouton?: value BP_Prog_Bouton_Lancer_Principale -> BP_Prog_Bouton_Lancer
- D?: value LED_Direction_Droite -> LED_Erreur
- R?: value ? -> 65
- U?: value Expender 2 -> Expander 2
- U?: value Expender 1 -> Expander 1
- U?: value Expender 3 -> Expander 3
Connections:
- net +3.3V: now also HDR1X5.VDD, ModeContinue/PasAPas?.NC, R?.2, U?.1 (VCC), U?.1 (VCC), U?.1 (VCC), U?.1 (VCC), U?.1 (VCC), U?.1 (VCC)
- net BP12: now also ModeContinue/PasAPas?.N
- net Earth: now also 100nF?.2, HDR1X5.VSS, ModeContinue/PasAPas?.NO, U?.4 (GND), U?.4 (GND), U?.4 (GND), U?.4 (GND), U?.4 (GND), U?.4 (GND)
- net at U=5V.1 (~{MCLR}/Vpp): now also R?.2
- net CKL1: now reaches U=5V.21 (RP10)
- net CKL1: now also U?.7 (CK1)
- net SDO1: now reaches U=5V.23 (RP12)
- net SDO1: now also U?.8 (SD1)
- net SDO2: now reaches U=5V.25 (RP14)
- net SDO2: now also U?.8 (SD1)
- net at U=5V.4 (RP0): now also HDR1X5.PGD
- net at U=5V.5 (RP1): now also HDR1X5.PGC
- net CKL2: now reaches U=5V.6 (SCK2OUT)
- net CKL2: now also U?.7 (CK1)
- net LED_ERREUR: no longer names the net of D?.2 (A), U=5V.11 (RP4)
- new net: U?.2 (CK0), U?.7 (CK1) (x4)
- new net: U?.5 (SD0), U?.8 (SD1) (x4)
- new net: 100nF?.1, HDR1X5.MCLR, R?.1, R?.1
Other:
- moved on the sheet: 100nF

Commit message: nvv eruebvue
Parts:
- removed Bouton?: BP_Prog_Etat_Apres_Valide, symbol Switch:SW_Push
- removed Bouton?: BP_Prog_Direction_SW, symbol Switch:SW_Push
- removed Bouton?: BP_Prog_Bouton_Lancer, symbol Switch:SW_Push
- removed Bouton?: BP_Prog_Etat_Avant_Letter, symbol Switch:SW_Push
- removed Bouton?: BP_Prog_Ecran_LCD_Moins, symbol Switch:SW_Push
- removed Bouton?: BP_Prog_Etat_Avant_Valide, symbol Switch:SW_Push
- removed Bouton?: BP_Prog_Etat_Avant_Plus, symbol Switch:SW_Push
- removed Bouton?: BP_Prog_Etat_Apres_Moins, symbol Switch:SW_Push
- removed Bouton?: BP_Prog_Ecran_LCD_Valide, symbol Switch:SW_Push
- removed Bouton?: BP_Prog_Etat_Avant_Moins, symbol Switch:SW_Push
- removed Bouton?: BP_Prog_Etat_Apres_Plus, symbol Switch:SW_Push
- removed R? (x8): 10k, symbol Device:R
- removed R? (x3): 4.7k, symbol Device:R
- added Bouton1: BP_Reset_Courant, symbol Switch:SW_Push
- added Bouton2: BP_Prog_Etat_Acceptation, symbol Switch:SW_Push
- added Bouton?: BP_Prog_Etat_Courant_Valide, symbol Switch:SW_Push
- added Bouton?: BP_Prog_Etat_Courant_Plus, symbol Switch:SW_Push
- added Bouton?: BP_Prog_Etat_Apres_Plus, symbol Switch:SW_Push
- added Bouton?: BP_Prog_Etat_Apres_Valide, symbol Switch:SW_Push
- added Bouton?: BP_Prog_Etat_Apres_Moins, symbol Switch:SW_Push
- added Bouton?: BP_Chg_Direction, symbol Switch:SW_Push
- added Bouton?: BP_Prog_Etat_Courant_Moins, symbol Switch:SW_Push
- added Bouton?: BP_Prog_Ecran_LCD_Valider, symbol Switch:SW_Push
- added Bouton?: BP_Lancer_Programme, symbol Switch:SW_Push
- added Bouton?: BP_Prog_Ecran_LCD_Moins, symbol Switch:SW_Push
- added R1, R2, R4, R5, R? (x10): 10k, symbol Device:R
- added R3, R? (x4): 65, symbol Device:R
- gave numbers to parts that had none: 1
Connections:
- net +3.3V: now also 100nF.1, 100nF.1, 100nF.2, 10µF.2, 7Seg1.5 (VSS), 7Seg2.5 (VSS), Bouton?.2, D?.1 (K), D?.1 (K), D?.1 (K), D?.4 (K), D?.4 (K), HDR1X5.VSS, ModeContinue/PasAPas?.NO, R?.1, R?.1, R?.2, U=5V.13 (VDD), U=5V.27 (VSS), U=5V.8 (VSS), U?.10 (VSS), U?.10 (VSS), U?.10 (VSS), U?.12 (SCK), U?.12 (SCK), U?.12 (SCK), U?.13 (SDA), U?.13 (SDA), U?.13 (SDA), U?.15 (A0), U?.16 (A1), U?.17 (A2), U?.17 (A2), U?.17 (A2), U?.2 (SCL), U?.3 (SDA), U?.4 (GND), U?.4 (GND), U?.4 (GND), U?.4 (GND), U?.4 (GND), U?.4 (GND), U?.4 (VSS), Bouton1.2, Bouton2.2, Bouton?.2, Bouton?.2, Bouton?.2, Bouton?.2, Bouton?.2, Bouton?.2, Bouton?.2, Bouton?.2, Bouton?.2, Bouton?.2, R1.1, R2.1, R4.2, R5.2, R?.2, R?.2, R?.2, R?.2, R?.2, R?.2, R?.2, R?.2, R?.2, R?.2; no longer Bouton?.1
- net BP1: now also Bouton?.1, R?.1
- net BP10: now also Bouton?.1, R?.1
- net BP11: now also Bouton?.1, R?.1
- net BP12: now also Bouton?.1, R?.1; no longer ModeContinue/PasAPas?.N
- net BP13: now also ModeContinue/PasAPas?.N
- net BP14: now also Bouton?.2, R?.2
- net BP15: now also Bouton?.2, R?.2; no longer Bouton?.2, R?.2
- net BP16: now also Bouton2.1, R5.1; no longer Bouton?.2, R?.2
- net BP2: now also Bouton?.1, R?.1
- net BP3: now also Bouton?.1, R?.1
- net BP4: now also Bouton1.1, R4.1
- net BP5: now also Bouton?.1, R?.1
- net BP6: now also Bouton?.1, R?.1
- net BP7: now also Bouton?.1, R?.1
- net BP8: now also Bouton?.1, R?.1
- net BP9: now also Bouton?.1, R?.1; no longer Bouton?.2, R?.2
- net LED2: now also R?.1; no longer D?.2 (GA)
- net LED3: now also R?.1; no longer D?.3 (BA)
- net LED6: now also R3.1; no longer D?.1 (RA)
- net LED7: now also R?.1; no longer D?.2 (GA)
- net LED8: now also R?.1; no longer D?.3 (BA)
- removed net Earth: 10µF.2, 7Seg1.5 (VSS), 7Seg2.5 (VSS), D?.1 (K), D?.1 (K), D?.1 (K), D?.4 (K), D?.4 (K), HDR1X5.VSS, ModeContinue/PasAPas?.NO, R?.1, R?.1, R?.1, U?.10 (VSS), U?.10 (VSS), U?.10 (VSS), U?.15 (A0), U?.16 (A1), U?.17 (A2), U?.17 (A2), U?.17 (A2), U?.4 (GND), U?.4 (GND), U?.4 (GND), U?.4 (GND), U?.4 (GND), U?.4 (GND), U?.4 (VSS)
- removed net SCL1: U=5V.17 (SCL1), U?.13 (SDA), U?.13 (SDA), U?.13 (SDA), U?.2 (SCL)
- removed net SDA1: U=5V.18 (SDA1), U?.12 (SCK), U?.12 (SCK), U?.12 (SCK), U?.3 (SDA)
- new net: R1.2, U=5V.17 (SCL1)
- new net: R2.2, U=5V.18 (SDA1)
- new net: D?.2 (GA), R?.2
- new net: D?.3 (BA), R?.2
